Commit message: Modified cell control pkg

File: src/robot_station_cell_control/urdf/robot_station_cell_controlled.urdf.xacro (robot description, xacro)
@@ -1,4 +1,4 @@
 <?xml version="1.0"?>
-<robot name="my_robot_cell" xmlns:xacro="http://ros.org/wiki/xacro">
+<robot name="robot_station_cell" xmlns:xacro="http://ros.org/wiki/xacro">
   <!--First, include the macro from our custom description-->
   <xacro:include filename="$(find robot_station_description)/urdf/common_properties.urdf"/>
@@ -8,11 +8,14 @@
   <!-- <xacro:include filename="$(find robot_station_description)/urdf/my_robot_cell_macro.xacro"/> -->
   <!--The driver already provides a control tag for the UR arm, we can directly include-->
-  <xacro:include filename="$(find ur_robot_driver)/urdf/ur.ros2_control.xacro"/>
+  <xacro:include filename="$(find ur_description)/urdf/ur.ros2_control.xacro"/>
   <!--We need to specify the arguments used for parametrizing our description-->
+  <!--Create a folder for wanted ur_type and copy those files from ur_description package in there; copied only ur20 files -->
+  <!--You could as well point to ur_description but this way you make sure you use the same files as start_robot.launch.py which searches in runtime_config_package for joint_limits.yaml, physical_parameters.yaml, visual_parameters.yaml and in description_package for default_kinematics.yaml (last one can be overwritten)-->
   <xacro:arg name="ur_type" default="ur10e"/>
-  <xacro:arg name="joint_limit_parameters_file" default="$(find ur_description)/config/$(arg ur_type)/joint_limits.yaml"/>
-  <xacro:arg name="kinematics_parameters_file" default="$(find ur_description)/config/$(arg ur_type)/default_kinematics.yaml"/>
-  <xacro:arg name="physical_parameters_file" default="$(find ur_description)/config/$(arg ur_type)/physical_parameters.yaml"/>
-  <xacro:arg name="visual_parameters_file" default="$(find ur_description)/config/$(arg ur_type)/visual_parameters.yaml"/>
+  <xacro:arg name="joint_limit_params" default="$(find robot_station_cell_control)/config/$(arg ur_type)/joint_limits.yaml"/>
+  <xacro:arg name="kinematics_params" default="$(find robot_station_cell_control)/config/$(arg ur_type)/default_kinematics.yaml"/>
+  <!-- <xacro:arg name="kinematics_params" default="$(find robot_station_cell_control)/config/my_robot_calibration.yaml"/> -->
+  <xacro:arg name="physical_params" default="$(find robot_station_cell_control)/config/$(arg ur_type)/physical_parameters.yaml"/>
+  <xacro:arg name="visual_params" default="$(find robot_station_cell_control)/config/$(arg ur_type)/visual_parameters.yaml"/>
   <xacro:arg name="robot_ip" default="0.0.0.0"/>
   <xacro:arg name="headless_mode" default="false" />
@@ -22,4 +25,7 @@
   <xacro:arg name="use_mock_hardware" default="false" />
   <xacro:arg name="mock_sensor_commands" default="false" />
+  <!--find hash_kinematics in kinematics_params-->
+  <xacro:property name="kinematics_params_file" value="$(arg kinematics_params)"/>
+  <xacro:property name="kinematics_hash" value="${xacro.load_yaml(kinematics_params_file)['kinematics']['hash']}"/>
   <link name="world" />
   <!--Create the scene description including the robot-->
@@ -43,11 +49,11 @@
     name="$(arg ur_type)"
     tf_prefix="$(arg ur_type)_"
-    kinematics_parameters_file="$(arg kinematics_parameters_file)"
+    hash_kinematics="${kinematics_hash}"
     robot_ip="$(arg robot_ip)"
     script_filename="$(arg ur_script_filename)"
     output_recipe_filename="$(arg ur_output_recipe_filename)"
     input_recipe_filename="$(arg ur_input_recipe_filename)"
-    use_mock_hardware="$(arg use_mock_hardware)"
-    mock_sensor_commands="$(arg mock_sensor_commands)"
+    use_fake_hardware="$(arg use_fake_hardware)"
+    fake_sensor_commands="$(arg fake_sensor_commands)"
     headless_mode="$(arg headless_mode)"
   />

Commit message: Added Bringup pkg

File: src/robot_station_cell_control/urdf/robot_station_cell_controlled.urdf.xacro (robot description, xacro)
@@ -6,4 +6,5 @@
   <xacro:include filename="$(find robot_station_description)/urdf/ur_orbbec_robotiq2f85_macro.urdf.xacro"/>
   <xacro:include filename="$(find robot_station_description)/urdf/messzelle_macro.urdf.xacro"/>
+  <xacro:include filename="$(find robot_station_description)/urdf/station_ur_orbbec_robotiq2f85_macro.urdf.xacro"/>
   <!-- <xacro:include filename="$(find robot_station_description)/urdf/my_robot_cell_macro.xacro"/> -->
   <!--The driver already provides a control tag for the UR arm, we can directly include-->
@@ -28,5 +29,5 @@
   <xacro:property name="kinematics_params_file" value="$(arg kinematics_params)"/>
   <xacro:property name="kinematics_hash" value="${xacro.load_yaml(kinematics_params_file)['kinematics']['hash']}"/>
-  <link name="world" />
+  <!-- <link name="world" /> -->
   <!--Create the scene description including the robot-->
   <!-- <xacro:my_robot_cell
@@ -40,9 +41,19 @@
     <origin xyz="0 0 1" rpy="0 0 0" />
   </xacro:my_robot_cell> -->
-  <xacro:robot_station_800x440 prefix="" parent="world" child="table_mount_link"/>
+  <!-- <xacro:robot_station_800x440 prefix="" parent="world" child="table_mount_link"/>
   <xacro:ur_orbbec_robotiq prefix="" parent="table_mount_link" finger_type="default" mount_orbbec="true">
       <origin xyz="0 0 0" rpy="0 0 ${pi/2}"/>
   </xacro:ur_orbbec_robotiq>
-  <xacro:messzelle_env prefix="" parent="world"/>
+  <xacro:messzelle_env prefix="" parent="world"/> -->
+  <xacro:station_ur_orbbec_robotiq
+      ur_type="ur10e"
+      tf_prefix=""
+      parent="world"
+      finger_type="default"
+      mount_orbbec="true"
+      include_station="true"
+      include_messzelle="true"
+      origin_xyz="0 0 0"
+      origin_rpy="0 0 ${pi/2}"/>
   <!--Create the control tag for the UR robot-->
   <xacro:ur_ros2_control

File: src/robot_station_cell_moveit_config/config/robot_station_cell.ros2_control.xacro (robot description, xacro)
@@ -50,4 +50,18 @@
                 <state_interface name="velocity"/>
             </joint>
+            <joint name="ct_left_door_joint">
+                <command_interface name="position"/>
+                <state_interface name="position">
+                  <param name="initial_value">${initial_positions['ct_left_door_joint']}</param>
+                </state_interface>
+                <state_interface name="velocity"/>
+            </joint>
+            <joint name="robotiq_85_left_knuckle_joint">
+                <command_interface name="position"/>
+                <state_interface name="position">
+                  <param name="initial_value">${initial_positions['robotiq_85_left_knuckle_joint']}</param>
+                </state_interface>
+                <state_interface name="velocity"/>
+            </joint>
         </ros2_control>
     </xacro:macro>

File: src/robot_station_cell_moveit_config/config/robot_station_cell.urdf.xacro (robot description, xacro)
@@ -1,9 +1,9 @@
 <?xml version="1.0"?>
 <robot xmlns:xacro="http://www.ros.org/wiki/xacro" name="robot_station_cell">
-    <xacro:arg name="initial_positions_file" default="initial_positions.yaml" />
+    <xacro:arg name="initial_positions_file2" default="initial_positions.yaml" />
     <!-- Import robot_station_cell urdf file -->
     <xacro:include filename="$(find robot_station_cell_control)/urdf/robot_station_cell_controlled.urdf.xacro" />
     <!-- Import control_xacro -->
     <xacro:include filename="robot_station_cell.ros2_control.xacro" />
-    <xacro:robot_station_cell_ros2_control name="FakeSystem" initial_positions_file="$(arg initial_positions_file)"/>
+    <xacro:robot_station_cell_ros2_control name="FakeSystem" initial_positions_file="$(arg initial_positions_file2)"/>
 </robot>

File: src/robot_station_description/urdf/station_ur_orbbec_robotiq2f85.urdf.xacro (robot description, xacro)
@@ -1,16 +1,21 @@
 <?xml version="1.0"?>
 <robot name="station_ur_orbbec_robotiq2f85" xmlns:xacro="http://wiki.ros.org/xacro">
-    <!-- Import the macro -->
-    <xacro:include filename="$(find robot_station_description)/urdf/station_ur_orbbec_robotiq2f85_macro.urdf.xacro"/>
-    <!-- Instantiate the complete station -->
-    <xacro:station_ur_orbbec_robotiq
-      ur_type="ur10e"
-      tf_prefix=""
-      parent="world"
-      finger_type="default"
-      mount_orbbec="true"
-      include_station="true"
-      include_messzelle="true"
-      origin_xyz="0 0 0"
-      origin_rpy="0 0 ${pi/2}"/>
+    <!-- Import macros -->
+    <xacro:include filename="$(find robot_station_description)/urdf/common_properties.urdf"/>
+    <xacro:include filename="$(find robot_station_description)/urdf/station_800x440_bosch_macro.urdf.xacro"/>
+    <xacro:include filename="$(find robot_station_description)/urdf/ur_orbbec_robotiq2f85_macro.urdf.xacro"/>
+    <xacro:include filename="$(find robot_station_description)/urdf/messzelle_macro.urdf.xacro"/>
+    <!-- <xacro:include filename="$(find ifl_air_description)/urdf/robotertisch_1520x900_macro.urdf.xacro"/> -->
+    <!-- <xacro:include filename="$(find ifl_air_description)/urdf/robotertisch_kameraaufsatz_macro.urdf.xacro"/> -->
+    <!-- <xacro:include filename="$(find ifl_air_description)/urdf/robotertisch_800x1400_macro.urdf.xacro"/> -->
+    <!-- <xacro:include filename="$(find ifl_air_description)/urdf/robotertisch_virtual_macro.urdf.xacro"/> -->
+    <!-- <xacro:include filename="$(find ifl_air_description)/urdf/roboter_oberdecke_macro.urdf.xacro"/> -->
+    <!-- create link fixed to the "world" -->
+    <link name="world" />
+    <!-- <xacro:arg name="joint_limit_params" default="$(find ifl_air_cell_small_ur_orbbec_robotiq_moveit_config)/config/joint_limits.yaml"/> -->
+    <xacro:robot_station_800x440 prefix="" parent="world" child="table_mount_link"/>
+    <xacro:ur_orbbec_robotiq prefix="" parent="table_mount_link" finger_type="default" mount_orbbec="true">
+        <origin xyz="0 0 0" rpy="0 0 ${pi/2}"/>
+    </xacro:ur_orbbec_robotiq>
+    <xacro:messzelle_env prefix="" parent="world"/>
 </robot>

File: src/robot_station_description/urdf/ur_orbbec_robotiq2f85_macro.urdf.xacro (robot description, xacro)
@@ -10,5 +10,5 @@
   <xacro:arg name="name" default="ur"/>
   <!-- Import macros -->
-  <xacro:include filename="$(find robotiq_description)/urdf/robotiq_2f_85_macro.urdf.xacro" />
+  <xacro:include filename="$(find robotiq_description)/urdf/robotiq_2f_140_macro.urdf.xacro" />
   <xacro:include filename="$(find robotiq_description)/urdf/robotiq_2f_85_75_macro.urdf.xacro" />
   <xacro:include filename="$(find robotiq_description)/urdf/robotiq_2f_85_160_macro.urdf.xacro" />
@@ -119,5 +119,5 @@
   <xacro:if value="${finger_type == 'default'}">
     <!-- Use the macro for original fingers -->
-    <xacro:robotiq_gripper name="Robotiq2f85OriginalFinger" prefix="${prefix}" parent="${prefix}gripper_base" use_fake_hardware="$(arg use_fake_hardware)">
+    <xacro:robotiq_gripper name="Robotiq2f140OriginalFinger" prefix="${prefix}" parent="${prefix}gripper_base" use_fake_hardware="$(arg use_fake_hardware)">
       <origin xyz="0 0 0" rpy="0 0 0" />
     </xacro:robotiq_gripper>
