Commit message: Adapt mqtt to the wbk environment

File: src/robot_station_description/urdf/messzelle_macro.urdf.xacro (robot description, xacro)
@@ -114,4 +114,5 @@
                     <mesh filename="package://robot_station_description/meshes/visual/table_simplified.stl"/>
                 </geometry>
+                <origin xyz="0 0 0" rpy="0 0 0" />
                 <material name="white"/>
             </visual>
@@ -120,5 +121,6 @@
                     <mesh filename="package://robot_station_description/meshes/visual/table_simplified.stl"/>
                 </geometry>
-            </collision>
+                <origin xyz="0 0 0" rpy="0 0 0" />
+            </collision>k
         </link>
         <joint name="${prefix}table_joint" type="fixed">

Commit message: Added cell_control and moveit_config packages

File: src/robot_station_description/urdf/messzelle_macro.urdf.xacro (robot description, xacro)
@@ -16,4 +16,5 @@
                 <origin xyz="0 0 0" rpy="0 0 0" />
             </collision>
+            <xacro:box_inertia m="10000.0" x="3.7" y="1.84" z="2.445" o_xyz="0 0 0" o_rpy="0 0 0"/>
         </link>
         <link name="${prefix}ct_left_door_link">
@@ -31,4 +32,5 @@
                 <origin xyz="0.25 0 0" rpy="0 0 0" />
             </collision>
+            <xacro:box_inertia m="5.0" x="0.5" y="0.02" z="1.84" o_xyz="0.25 0 0" o_rpy="0 0 0"/>
         </link>
         <link name="${prefix}ct_right_door_link">
@@ -46,14 +48,15 @@
                 <origin xyz="-0.25 0 0" rpy="0 0 0" />
             </collision>
+            <xacro:box_inertia m="5.0" x="0.5" y="0.02" z="1.84" o_xyz="-0.25 0 0" o_rpy="0 0 0"/>
         </link>
         <joint name="${prefix}ct_machine_joint" type="fixed">
             <parent link="${parent}"/>
             <child link="${prefix}ct_base_link"/>
-            <origin xyz="0 0 0" rpy="0 0 0" />
+            <origin xyz="1.8 0.92 1.2225" rpy="0 0 0" />
         </joint>
         <joint name="${prefix}ct_left_door_joint" type="prismatic">
             <parent link="${prefix}ct_base_link"/>
             <child link="${prefix}ct_left_door_link"/>
-            <origin xyz="1.445 1.84 1.22" rpy="0 0 0" />
+            <origin xyz="-0.405 0.92 -0.0025" rpy="0 0 0" />
             <axis xyz="1 0 0"/>
             <limit lower="0" upper="0.5" effort="1000" velocity="1.0"/>
@@ -62,5 +65,5 @@
             <parent link="${prefix}ct_base_link"/>
             <child link="${prefix}ct_right_door_link"/>
-            <origin xyz="1.445 1.84 1.22" rpy="0 0 0" />
+            <origin xyz="-0.405 0.92 -0.0025" rpy="0 0 0" />
             <axis xyz="-1 0 0"/>
             <limit lower="0" upper="0.5" effort="1000" velocity="1.0"/>
@@ -81,4 +84,5 @@
                 <origin xyz="0 0 0" rpy="0 0 0" />
             </collision>
+            <xacro:box_inertia m="50.0" x="0.1" y="4.865" z="3.65" o_xyz="0 0 0" o_rpy="0 0 0"/>
         </link>
         <link name="${prefix}slide_window_link">
@@ -96,12 +100,13 @@
                 <origin xyz="0 0 0" rpy="0 0 ${pi/2.0}" />
             </collision>
+            <xacro:box_inertia m="5.0" x="1.45" y="0.1" z="1.0" o_xyz="0 0 0" o_rpy="0 0 ${pi/2.0}"/>
         </link>
         <joint name="${prefix}wall1_joint" type="fixed">
             <parent link="${parent}"/>
             <child link="${prefix}wall1_link"/>
-            <origin xyz="0 0 0" rpy="0 0 0" />
+            <origin xyz="-0.05 2.4325 1.825" rpy="0 0 0" />
         </joint>
         <joint name="${prefix}slide_window_joint" type="prismatic">
-            <parent link="${prefix}wall1_link"/>
+            <parent link="${parent}"/>
             <child link="${prefix}slide_window_link"/>
             <origin xyz="0.0 2.712 1.5" rpy="0 0 0" />
@@ -122,10 +127,11 @@
                 </geometry>
                 <origin xyz="0 0 0" rpy="0 0 0" />
-            </collision>k
+            </collision>
+            <xacro:box_inertia m="5.0" x="1.5" y="0.8" z="1.0" o_xyz="0 0 0" o_rpy="0 0 0"/>
         </link>
         <joint name="${prefix}table_joint" type="fixed">
             <parent link="${parent}"/>
             <child link="${prefix}table_link"/>
-            <origin xyz="2.95 2.34 0" rpy="0 0 0" />
+            <origin xyz="2.95 2.34 0.5" rpy="0 0 0" />
         </joint>
     </xacro:macro>

File: src/robot_station_description/urdf/station_800x440_bosch_macro.urdf.xacro (robot description, xacro)
@@ -16,9 +16,5 @@
           </geometry>
         </collision>
-        <!-- <inertial>
-          <mass value="2" />
-          <origin xyz="0 0 0" />
-          <inertia ixx="8.432e-3" ixy="3.804169e-6" ixz="7.00981e-7" iyy="8.460e-3" iyz="-8.41529e-7" izz="1.606e-2" />
-        </inertial> -->
+        <xacro:box_inertia m="150.0" x="0.8" y="0.44" z="0.848" o_xyz="0 0 0" o_rpy="0 0 0"/>
     </link>
     <joint name="${prefix}station_800x440_base_joint" type="fixed">

Commit message: urdf and moveit config with robotiq 2f_140

File: src/robot_station_description/urdf/messzelle_macro.urdf.xacro (robot description, xacro)
@@ -49,4 +49,52 @@
             </collision>
             <xacro:box_inertia m="5.0" x="0.5" y="0.02" z="1.84" o_xyz="-0.25 0 0" o_rpy="0 0 0"/>
+        </link>
+        <link name="${prefix}ct_load_workbench_link">
+            <visual>
+                <geometry>
+                    <box size="0.345 0.46 0.30" />
+                </geometry>
+                <material name="grey" />
+                <origin xyz="0 0 0" rpy="0 0 0" />
+            </visual>
+            <collision>
+                <geometry>
+                    <box size="0.345 0.46 0.30" />
+                </geometry>
+                <origin xyz="0 0 0" rpy="0 0 0" />
+            </collision>
+            <xacro:box_inertia m="2.0" x="0.345" y="0.46" z="0.30" o_xyz="0 0 0" o_rpy="0 0 0"/>
+        </link>
+        <link name="${prefix}ct_load_disk_link">
+            <visual>
+                <geometry>
+                    <cylinder radius="0.15" length="0.05" />
+                </geometry>
+                <material name="grey" />
+                <origin xyz="0 0 0" rpy="0 0 0" />
+            </visual>
+            <collision>
+                <geometry>
+                    <cylinder radius="0.15" length="0.05" />
+                </geometry>
+                <origin xyz="0 0 0" rpy="0 0 0" />
+            </collision>
+            <xacro:cylinder_inertia m="1.0" r="0.15" l="0.05" o_xyz="0 0 0" o_rpy="0 0 0"/>
+        </link>
+        <link name="${prefix}ct_load_block_link">
+            <visual>
+                <geometry>
+                    <box size="0.1 0.3 0.34" />
+                </geometry>
+                <material name="grey" />
+                <origin xyz="0 0 0" rpy="0 0 0" />
+            </visual>
+            <collision>
+                <geometry>
+                    <box size="0.1 0.3 0.34" />
+                </geometry>
+                <origin xyz="0 0 0" rpy="0 0 0" />
+            </collision>
+            <xacro:box_inertia m="1.0" x="0.1" y="0.3" z="0.34" o_xyz="0 0 0" o_rpy="0 0 0"/>
         </link>
         <joint name="${prefix}ct_machine_joint" type="fixed">
@@ -70,4 +118,19 @@
             <mimic joint="${prefix}ct_left_door_joint" multiplier="1.0" offset="0.0" />
         </joint>
+        <joint name="${prefix}ct_load_workbench_joint" type="fixed">
+            <parent link="${prefix}ct_base_link"/>
+            <child link="${prefix}ct_load_workbench_link"/>
+            <origin xyz="-0.405 0.49 -0.3655" rpy="0 0 0" />
+        </joint>
+        <joint name="${prefix}ct_load_disk_joint" type="fixed">
+            <parent link="${prefix}ct_load_workbench_link"/>
+            <child link="${prefix}ct_load_disk_link"/>
+            <origin xyz="0.0 -0.05 0.069" rpy="0 0 0" />
+        </joint>
+        <joint name="${prefix}ct_load_block_joint" type="fixed">
+            <parent link="${prefix}ct_load_disk_link"/>
+            <child link="${prefix}ct_load_block_link"/>
+            <origin xyz="0.0 0.0 0.195" rpy="0 0 0" />
+        </joint>
         <link name="${prefix}wall1_link">
             <visual>

File: src/robot_station_description/urdf/ur_orbbec_robotiq2f85_macro.urdf.xacro (robot description, xacro)
@@ -11,5 +11,6 @@
   <!-- Import macros -->
   <xacro:include filename="$(find robotiq_description)/urdf/robotiq_2f_140_macro.urdf.xacro" />
-  <!-- <xacro:include filename="$(find robotiq_description)/urdf/robotiq_2f_85_75_macro.urdf.xacro" />
+  <!-- <xacro:include filename="$(find robotiq_description)/urdf/robotiq_2f_85_macro.urdf.xacro" />
+  <xacro:include filename="$(find robotiq_description)/urdf/robotiq_2f_85_75_macro.urdf.xacro" />
   <xacro:include filename="$(find robotiq_description)/urdf/robotiq_2f_85_160_macro.urdf.xacro" /> -->
   <xacro:include filename="$(find ur_description)/urdf/ur_macro.xacro"/>
@@ -78,5 +79,26 @@
     safety_limits="$(arg safety_limits)"
     safety_pos_margin="$(arg safety_pos_margin)"
-    safety_k_position="$(arg safety_k_position)" >
+    safety_k_position="$(arg safety_k_position)"
+    headless_mode="$(arg headless_mode)"
+    robot_ip="$(arg robot_ip)"
+    script_filename="$(arg script_filename)"
+    output_recipe_filename="$(arg output_recipe_filename)"
+    input_recipe_filename="$(arg input_recipe_filename)"
+    use_tool_communication="$(arg use_tool_communication)"
+    tool_voltage="$(arg tool_voltage)"
+    tool_parity="$(arg tool_parity)"
+    tool_baud_rate="$(arg tool_baud_rate)"
+    tool_stop_bits="$(arg tool_stop_bits)"
+    tool_rx_idle_chars="$(arg tool_rx_idle_chars)"
+    tool_tx_idle_chars="$(arg tool_tx_idle_chars)"
+    tool_device_name="$(arg tool_device_name)"
+    tool_tcp_port="$(arg tool_tcp_port)"
+    reverse_ip="$(arg reverse_ip)"
+    script_command_port="$(arg script_command_port)"
+    reverse_port="$(arg reverse_port)"
+    script_sender_port="$(arg script_sender_port)"
+    trajectory_port="$(arg trajectory_port)"
+    use_fake_hardware="$(arg use_fake_hardware)"
+    fake_sensor_commands="$(arg fake_sensor_commands)" >
     <origin xyz="0 0 0" rpy="0 0 0" />
     <!-- position robot in the world -->

File: src/robot_station_moveit_config/config/station_ur_orbbec_robotiq2f85.ros2_control.xacro (robot description, xacro)
@@ -50,18 +50,4 @@
                 <state_interface name="velocity"/>
             </joint>
-            <joint name="ct_left_door_joint">
-                <command_interface name="position"/>
-                <state_interface name="position">
-                  <param name="initial_value">${initial_positions['ct_left_door_joint']}</param>
-                </state_interface>
-                <state_interface name="velocity"/>
-            </joint>
-            <joint name="slide_window_joint">
-                <command_interface name="position"/>
-                <state_interface name="position">
-                  <param name="initial_value">${initial_positions['slide_window_joint']}</param>
-                </state_interface>
-                <state_interface name="velocity"/>
-            </joint>
             <joint name="finger_joint">
                 <command_interface name="position"/>
