Commit message: Convert description file to macro to spawn the robot station

File: src/robot_station_description/urdf/station_ur_orbbec_robotiq2f85.urdf.xacro (robot description, xacro)
@@ -1,21 +1,16 @@
 <?xml version="1.0"?>
 <robot name="station_ur_orbbec_robotiq2f85" xmlns:xacro="http://wiki.ros.org/xacro">
-    <!-- Import macros -->
-    <xacro:include filename="$(find robot_station_description)/urdf/common_properties.urdf"/>
-    <xacro:include filename="$(find robot_station_description)/urdf/station_800x440_bosch_macro.urdf.xacro"/>
-    <xacro:include filename="$(find robot_station_description)/urdf/ur_orbbec_robotiq2f85_macro.urdf.xacro"/>
-    <xacro:include filename="$(find robot_station_description)/urdf/messzelle_macro.urdf.xacro"/>
-    <!-- <xacro:include filename="$(find ifl_air_description)/urdf/robotertisch_1520x900_macro.urdf.xacro"/> -->
-    <!-- <xacro:include filename="$(find ifl_air_description)/urdf/robotertisch_kameraaufsatz_macro.urdf.xacro"/> -->
-    <!-- <xacro:include filename="$(find ifl_air_description)/urdf/robotertisch_800x1400_macro.urdf.xacro"/> -->
-    <!-- <xacro:include filename="$(find ifl_air_description)/urdf/robotertisch_virtual_macro.urdf.xacro"/> -->
-    <!-- <xacro:include filename="$(find ifl_air_description)/urdf/roboter_oberdecke_macro.urdf.xacro"/> -->
-    <!-- create link fixed to the "world" -->
-    <link name="world" />
-    <!-- <xacro:arg name="joint_limit_params" default="$(find ifl_air_cell_small_ur_orbbec_robotiq_moveit_config)/config/joint_limits.yaml"/> -->
-    <xacro:robot_station_800x440 prefix="" parent="world" child="table_mount_link"/>
-    <xacro:ur_orbbec_robotiq prefix="" parent="table_mount_link" finger_type="default" mount_orbbec="true">
-        <origin xyz="0 0 0" rpy="0 0 ${pi/2}"/>
-    </xacro:ur_orbbec_robotiq>
-    <xacro:messzelle_env prefix="" parent="world"/>
+    <!-- Import the macro -->
+    <xacro:include filename="$(find robot_station_description)/urdf/station_ur_orbbec_robotiq2f85_macro.urdf.xacro"/>
+    <!-- Instantiate the complete station -->
+    <xacro:station_ur_orbbec_robotiq
+      ur_type="ur10e"
+      tf_prefix=""
+      parent="world"
+      finger_type="default"
+      mount_orbbec="true"
+      include_station="true"
+      include_messzelle="true"
+      origin_xyz="0 0 0"
+      origin_rpy="0 0 ${pi/2}"/>
 </robot>

Commit message: Modified Moveit Config

File: src/robot_station_description/urdf/station_ur_orbbec_robotiq2f85.urdf.xacro (robot description, xacro)
@@ -13,5 +13,5 @@
     <!-- create link fixed to the "world" -->
     <link name="world" />
-    <!-- <xacro:arg name="joint_limit_params" default="$(find ifl_air_cell_small_ur_orbbec_robotiq_moveit_config)/config/joint_limits.yaml"/> -->
+    <!-- <xacro:arg name="joint_limit_params" default="$(find robot_station_cell_moveit_config)/config/joint_limits.yaml"/> -->
     <xacro:robot_station_800x440 prefix="" parent="world" child="table_mount_link"/>
     <xacro:ur_orbbec_robotiq prefix="" parent="table_mount_link" finger_type="default" mount_orbbec="true">

File: src/robot_station_description/urdf/station_ur_orbbec_robotiq2f85_macro.urdf.xacro (robot description, xacro)
@@ -22,9 +22,4 @@
     origin_xyz:='0 0 0'
     origin_rpy:='0 0 0'">
-    <!-- Import common properties and macros -->
-    <xacro:include filename="$(find robot_station_description)/urdf/common_properties.urdf"/>
-    <xacro:include filename="$(find robot_station_description)/urdf/station_800x440_bosch_macro.urdf.xacro"/>
-    <xacro:include filename="$(find robot_station_description)/urdf/ur_orbbec_robotiq2f85_macro.urdf.xacro"/>
-    <xacro:include filename="$(find robot_station_description)/urdf/messzelle_macro.urdf.xacro"/>
     <!-- Create world link if parent is "world" -->
     <xacro:if value="${parent == 'world'}">

File: src/robot_station_description/urdf/ur_orbbec_robotiq2f85_macro.urdf.xacro (robot description, xacro)
@@ -11,6 +11,6 @@
   <!-- Import macros -->
   <xacro:include filename="$(find robotiq_description)/urdf/robotiq_2f_140_macro.urdf.xacro" />
-  <xacro:include filename="$(find robotiq_description)/urdf/robotiq_2f_85_75_macro.urdf.xacro" />
-  <xacro:include filename="$(find robotiq_description)/urdf/robotiq_2f_85_160_macro.urdf.xacro" />
+  <!-- <xacro:include filename="$(find robotiq_description)/urdf/robotiq_2f_85_75_macro.urdf.xacro" />
+  <xacro:include filename="$(find robotiq_description)/urdf/robotiq_2f_85_160_macro.urdf.xacro" /> -->
   <xacro:include filename="$(find ur_description)/urdf/ur_macro.xacro"/>
   <xacro:include filename="$(find robotiq_description)/urdf/ur_to_robotiq_adapter.urdf.xacro"/>
@@ -91,30 +91,4 @@
   <xacro:ur_to_robotiq prefix="${prefix}" parent="${prefix}tool0_ext" child="${prefix}gripper_base" rotation="${pi/2}"/>
   <!-- gripper -->
-  <xacro:if value="${finger_type == 'custom_160'}">
-    <!-- Use the macro for 160mm fingers -->
-    <xacro:robotiq_gripper_160 name="Robotiq2f85Finger160" prefix="${prefix}" parent="${prefix}gripper_base" use_fake_hardware="$(arg use_fake_hardware)">
-      <origin xyz="0 0 0" rpy="0 0 0" />
-    </xacro:robotiq_gripper_160>
-    <!--- tcp frame-->
-    <joint name="${prefix}tool0_to_tcp" type="fixed">
-        <parent link="${prefix}tool0"/>
-        <child link="tcp"/>
-        <origin xyz="0 0 0.303" rpy="0 0 0"/>
-    </joint>
-    <link name="tcp"/>
-  </xacro:if>
-  <xacro:if value="${finger_type == 'custom_75'}">
-    <!-- Use the macro for 75mm fingers -->
-    <xacro:robotiq_gripper_75 name="Robotiq2f85Finger75" prefix="${prefix}" parent="${prefix}gripper_base" use_fake_hardware="$(arg use_fake_hardware)">
-      <origin xyz="0 0 0" rpy="0 0 0" />
-    </xacro:robotiq_gripper_75>
-    <!--- tcp frame-->
-    <joint name="${prefix}tool0_to_tcp" type="fixed">
-        <parent link="${prefix}tool0"/>
-        <child link="tcp"/>
-        <origin xyz="0 0 0.218" rpy="0 0 0"/>
-    </joint>
-    <link name="tcp"/>
-  </xacro:if>
   <xacro:if value="${finger_type == 'default'}">
     <!-- Use the macro for original fingers -->

File: src/robot_station_moveit_config/config/station_ur_orbbec_robotiq2f85.ros2_control.xacro (robot description, xacro)
@@ -50,4 +50,25 @@
                 <state_interface name="velocity"/>
             </joint>
+            <joint name="ct_left_door_joint">
+                <command_interface name="position"/>
+                <state_interface name="position">
+                  <param name="initial_value">${initial_positions['ct_left_door_joint']}</param>
+                </state_interface>
+                <state_interface name="velocity"/>
+            </joint>
+            <joint name="slide_window_joint">
+                <command_interface name="position"/>
+                <state_interface name="position">
+                  <param name="initial_value">${initial_positions['slide_window_joint']}</param>
+                </state_interface>
+                <state_interface name="velocity"/>
+            </joint>
+            <joint name="finger_joint">
+                <command_interface name="position"/>
+                <state_interface name="position">
+                  <param name="initial_value">${initial_positions['finger_joint']}</param>
+                </state_interface>
+                <state_interface name="velocity"/>
+            </joint>
         </ros2_control>
     </xacro:macro>

Commit message: Request to merge dev branch to main (#1)
* modified moveit config

* Convert description file to macro to spawn the robot station

* Updated moveit config

* Added Bringup pkg

* Modified Moveit Config

* urdf and moveit config with robotiq 2f_140

* Updated Moveit launch file and configuration

* Removed robotiq_2f_urcap_adapter submodule reference and temp files

---------

Co-authored-by: YiminHu26 <yimin.hu@student.kit.edu>

File: src/robot_station_description/urdf/station_ur_orbbec_robotiq2f85.urdf.xacro (robot description, xacro)
@@ -13,5 +13,5 @@
     <!-- create link fixed to the "world" -->
     <link name="world" />
-    <!-- <xacro:arg name="joint_limit_params" default="$(find ifl_air_cell_small_ur_orbbec_robotiq_moveit_config)/config/joint_limits.yaml"/> -->
+    <!-- <xacro:arg name="joint_limit_params" default="$(find robot_station_cell_moveit_config)/config/joint_limits.yaml"/> -->
     <xacro:robot_station_800x440 prefix="" parent="world" child="table_mount_link"/>
     <xacro:ur_orbbec_robotiq prefix="" parent="table_mount_link" finger_type="default" mount_orbbec="true">

File: src/robot_station_description/urdf/ur_orbbec_robotiq2f85_macro.urdf.xacro (robot description, xacro)
@@ -10,7 +10,8 @@
   <xacro:arg name="name" default="ur"/>
   <!-- Import macros -->
-  <xacro:include filename="$(find robotiq_description)/urdf/robotiq_2f_85_macro.urdf.xacro" />
+  <xacro:include filename="$(find robotiq_description)/urdf/robotiq_2f_140_macro.urdf.xacro" />
+  <!-- <xacro:include filename="$(find robotiq_description)/urdf/robotiq_2f_85_macro.urdf.xacro" />
   <xacro:include filename="$(find robotiq_description)/urdf/robotiq_2f_85_75_macro.urdf.xacro" />
-  <xacro:include filename="$(find robotiq_description)/urdf/robotiq_2f_85_160_macro.urdf.xacro" />
+  <xacro:include filename="$(find robotiq_description)/urdf/robotiq_2f_85_160_macro.urdf.xacro" /> -->
   <xacro:include filename="$(find ur_description)/urdf/ur_macro.xacro"/>
   <xacro:include filename="$(find robotiq_description)/urdf/ur_to_robotiq_adapter.urdf.xacro"/>
@@ -78,5 +79,26 @@
     safety_limits="$(arg safety_limits)"
     safety_pos_margin="$(arg safety_pos_margin)"
-    safety_k_position="$(arg safety_k_position)" >
+    safety_k_position="$(arg safety_k_position)"
+    headless_mode="$(arg headless_mode)"
+    robot_ip="$(arg robot_ip)"
+    script_filename="$(arg script_filename)"
+    output_recipe_filename="$(arg output_recipe_filename)"
+    input_recipe_filename="$(arg input_recipe_filename)"
+    use_tool_communication="$(arg use_tool_communication)"
+    tool_voltage="$(arg tool_voltage)"
+    tool_parity="$(arg tool_parity)"
+    tool_baud_rate="$(arg tool_baud_rate)"
+    tool_stop_bits="$(arg tool_stop_bits)"
+    tool_rx_idle_chars="$(arg tool_rx_idle_chars)"
+    tool_tx_idle_chars="$(arg tool_tx_idle_chars)"
+    tool_device_name="$(arg tool_device_name)"
+    tool_tcp_port="$(arg tool_tcp_port)"
+    reverse_ip="$(arg reverse_ip)"
+    script_command_port="$(arg script_command_port)"
+    reverse_port="$(arg reverse_port)"
+    script_sender_port="$(arg script_sender_port)"
+    trajectory_port="$(arg trajectory_port)"
+    use_fake_hardware="$(arg use_fake_hardware)"
+    fake_sensor_commands="$(arg fake_sensor_commands)" >
     <origin xyz="0 0 0" rpy="0 0 0" />
     <!-- position robot in the world -->
@@ -91,33 +113,7 @@
   <xacro:ur_to_robotiq prefix="${prefix}" parent="${prefix}tool0_ext" child="${prefix}gripper_base" rotation="${pi/2}"/>
   <!-- gripper -->
-  <xacro:if value="${finger_type == 'custom_160'}">
-    <!-- Use the macro for 160mm fingers -->
-    <xacro:robotiq_gripper_160 name="Robotiq2f85Finger160" prefix="${prefix}" parent="${prefix}gripper_base" use_fake_hardware="$(arg use_fake_hardware)">
-      <origin xyz="0 0 0" rpy="0 0 0" />
-    </xacro:robotiq_gripper_160>
-    <!--- tcp frame-->
-    <joint name="${prefix}tool0_to_tcp" type="fixed">
-        <parent link="${prefix}tool0"/>
-        <child link="tcp"/>
-        <origin xyz="0 0 0.303" rpy="0 0 0"/>
-    </joint>
-    <link name="tcp"/>
-  </xacro:if>
-  <xacro:if value="${finger_type == 'custom_75'}">
-    <!-- Use the macro for 75mm fingers -->
-    <xacro:robotiq_gripper_75 name="Robotiq2f85Finger75" prefix="${prefix}" parent="${prefix}gripper_base" use_fake_hardware="$(arg use_fake_hardware)">
-      <origin xyz="0 0 0" rpy="0 0 0" />
-    </xacro:robotiq_gripper_75>
-    <!--- tcp frame-->
-    <joint name="${prefix}tool0_to_tcp" type="fixed">
-        <parent link="${prefix}tool0"/>
-        <child link="tcp"/>
-        <origin xyz="0 0 0.218" rpy="0 0 0"/>
-    </joint>
-    <link name="tcp"/>
-  </xacro:if>
   <xacro:if value="${finger_type == 'default'}">
     <!-- Use the macro for original fingers -->
-    <xacro:robotiq_gripper name="Robotiq2f85OriginalFinger" prefix="${prefix}" parent="${prefix}gripper_base" use_fake_hardware="$(arg use_fake_hardware)">
+    <xacro:robotiq_gripper name="Robotiq2f140OriginalFinger" prefix="${prefix}" parent="${prefix}gripper_base" use_fake_hardware="$(arg use_fake_hardware)">
       <origin xyz="0 0 0" rpy="0 0 0" />
     </xacro:robotiq_gripper>

File: src/robot_station_moveit_config/config/station_ur_orbbec_robotiq2f85.ros2_control.xacro (robot description, xacro)
@@ -50,4 +50,11 @@
                 <state_interface name="velocity"/>
             </joint>
+            <joint name="finger_joint">
+                <command_interface name="position"/>
+                <state_interface name="position">
+                  <param name="initial_value">${initial_positions['finger_joint']}</param>
+                </state_interface>
+                <state_interface name="velocity"/>
+            </joint>
         </ros2_control>
     </xacro:macro>
