Commit message: Change name 2f_85 to 2f_140

File: src/robot_station_description/urdf/station_ur_orbbec_robotiq2f140.urdf.xacro (robot description, xacro)
@@ -1,8 +1,8 @@
 <?xml version="1.0"?>
-<robot name="station_ur_orbbec_robotiq2f85" xmlns:xacro="http://wiki.ros.org/xacro">
+<robot name="station_ur_orbbec_robotiq2f140" xmlns:xacro="http://wiki.ros.org/xacro">
     <!-- Import macros -->
     <xacro:include filename="$(find robot_station_description)/urdf/common_properties.urdf"/>
     <xacro:include filename="$(find robot_station_description)/urdf/station_800x440_bosch_macro.urdf.xacro"/>
-    <xacro:include filename="$(find robot_station_description)/urdf/ur_orbbec_robotiq2f85_macro.urdf.xacro"/>
+    <xacro:include filename="$(find robot_station_description)/urdf/ur_orbbec_robotiq2f140_macro.urdf.xacro"/>
     <xacro:include filename="$(find robot_station_description)/urdf/messzelle_macro.urdf.xacro"/>
     <!-- <xacro:include filename="$(find ifl_air_description)/urdf/robotertisch_1520x900_macro.urdf.xacro"/> -->

File: src/robot_station_moveit_config/config/station_ur_orbbec_robotiq2f140.ros2_control.xacro (robot description, xacro)
@@ -1,5 +1,5 @@
 <?xml version="1.0"?>
 <robot xmlns:xacro="http://www.ros.org/wiki/xacro">
-    <xacro:macro name="station_ur_orbbec_robotiq2f85_ros2_control" params="name initial_positions_file">
+    <xacro:macro name="station_ur_orbbec_robotiq2f140_ros2_control" params="name initial_positions_file">
         <xacro:property name="initial_positions" value="${load_yaml(initial_positions_file)['initial_positions']}"/>
         <ros2_control name="${name}" type="system">

Commit message: Adjusted moveit config

File: src/robot_station_description/urdf/station_ur_orbbec_robotiq2f140.urdf.xacro (robot description, xacro)
@@ -16,5 +16,5 @@
     <xacro:robot_station_800x440 prefix="" parent="world" child="table_mount_link"/>
     <xacro:ur_orbbec_robotiq prefix="" parent="table_mount_link" finger_type="default" mount_orbbec="true">
-        <origin xyz="0 0 0" rpy="0 0 ${pi/2}"/>
+        <origin xyz="0 0 0" rpy="0 0 0"/>
     </xacro:ur_orbbec_robotiq>
     <xacro:messzelle_env prefix="" parent="world"/>

File: src/robot_station_description/urdf/ur_orbbec_robotiq2f140_macro.urdf.xacro (robot description, xacro)
@@ -101,5 +101,5 @@
     use_fake_hardware="$(arg use_fake_hardware)"
     fake_sensor_commands="$(arg fake_sensor_commands)" >
-    <origin xyz="0 0 0" rpy="0 0 0" />
+    <origin xyz="0 0 0" rpy="0 0 -${pi/2}" />
     <!-- position robot in the world -->
   </xacro:ur_robot>

Commit message: Added AGV Table in description and moveit config

File: src/robot_station_description/urdf/station_ur_orbbec_robotiq2f140.urdf.xacro (robot description, xacro)
@@ -4,4 +4,5 @@
     <xacro:include filename="$(find robot_station_description)/urdf/common_properties.urdf"/>
     <xacro:include filename="$(find robot_station_description)/urdf/station_800x440_bosch_macro.urdf.xacro"/>
+    <xacro:include filename="$(find robot_station_description)/urdf/agv_station_550x400_macro.urdf.xacro"/>
     <xacro:include filename="$(find robot_station_description)/urdf/ur_orbbec_robotiq2f140_macro.urdf.xacro"/>
     <xacro:include filename="$(find robot_station_description)/urdf/messzelle_macro.urdf.xacro"/>
@@ -15,4 +16,5 @@
     <!-- <xacro:arg name="joint_limit_params" default="$(find robot_station_cell_moveit_config)/config/joint_limits.yaml"/> -->
     <xacro:robot_station_800x440 prefix="" parent="world" child="table_mount_link"/>
+    <xacro:agv_station_550x400 prefix="" parent="world" />
     <xacro:ur_orbbec_robotiq prefix="" parent="table_mount_link" finger_type="default" mount_orbbec="true">
         <origin xyz="0 0 0" rpy="0 0 0"/>

File: src/robot_station_description/urdf/ur_orbbec_robotiq2f140_macro.urdf.xacro (robot description, xacro)
@@ -122,5 +122,5 @@
         <parent link="${prefix}tool0"/>
         <child link="tcp"/>
-        <origin xyz="0 0 0.18" rpy="0 0 0"/>
+        <origin xyz="0 0 0.23" rpy="0 0 0"/>
     </joint>
     <link name="tcp"/>
