Commit message: Updated URDF

File: src/robot_station_description/urdf/messzelle_new_macro.urdf.xacro (robot description, xacro)
@@ -107,4 +107,5 @@
                 <mesh filename="package://robot_station_description/meshes/collision/ct_load_block.stl"
                 scale="0.001 0.001 0.001" />
+                <origin xyz="0 0 0" rpy="0 0 0" />
             </collision>
         </link>

Commit message: Updated collision tag of ct_load_block_link

File: src/robot_station_description/urdf/messzelle_new_macro.urdf.xacro (robot description, xacro)
@@ -101,10 +101,11 @@
                     scale="0.001 0.001 0.001" />
                 </geometry>
-                <material name="grey" />
-                <origin xyz="0 0 0" rpy="0 0 0" />
-            </visual>
-            <collision>
-                <mesh filename="package://robot_station_description/meshes/collision/ct_load_block.stl"
-                scale="0.001 0.001 0.001" />
+                <origin xyz="0 0 0" rpy="0 0 0" />
+            </visual>
+            <collision>
+                <geometry>
+                    <mesh filename="package://robot_station_description/meshes/collision/ct_load_block.stl"
+                    scale="0.001 0.001 0.001" />
+                </geometry>
                 <origin xyz="0 0 0" rpy="0 0 0" />
             </collision>

Commit message: Adapted axis on ct_load_block to angle grinder axis

File: src/robot_station_description/urdf/messzelle_new_macro.urdf.xacro (robot description, xacro)
@@ -150,5 +150,5 @@
             <parent link="${prefix}ct_load_block_link"/>
             <child link="${prefix}placement_link"/>
-            <origin xyz="0.0 0.15 0.17" rpy="0 0 0" />
+            <origin xyz="0.0 0.15 0.17" rpy="0 -${pi/4} ${3*pi/2}" />
         </joint>
         <link name="${prefix}wall1_link">

Commit message: Test setup, modified param in description and moveit config

File: src/robot_station_description/urdf/messzelle_new_macro.urdf.xacro (robot description, xacro)
@@ -103,5 +103,5 @@
                 <origin xyz="0 0 0" rpy="0 0 0" />
             </visual>
-            <collision>
+            <!-- <collision>
                 <geometry>
                     <mesh filename="package://robot_station_description/meshes/collision/ct_load_block.stl"
@@ -109,5 +109,5 @@
                 </geometry>
                 <origin xyz="0 0 0" rpy="0 0 0" />
-            </collision>
+            </collision> -->
         </link>
         <link name="${prefix}placement_link" />
@@ -135,5 +135,5 @@
             <parent link="${prefix}ct_base_link"/>
             <child link="${prefix}ct_load_workbench_link"/>
-            <origin xyz="-0.405 0.49 -0.3655" rpy="0 0 0" />
+            <origin xyz="-0.405 0.49 -0.4135" rpy="0 0 0" />
         </joint>
         <joint name="${prefix}ct_load_disk_joint" type="fixed">
@@ -150,5 +150,5 @@
             <parent link="${prefix}ct_load_block_link"/>
             <child link="${prefix}placement_link"/>
-            <origin xyz="0.0 0.15 0.17" rpy="0 -${pi/4} ${3*pi/2}" />
+            <origin xyz="0.0 0.16 0.15" rpy="0 -${pi/4} ${3*pi/2}" />
         </joint>
         <link name="${prefix}wall1_link">

Commit message: Offset placement link, top down view from camera for experiments 20260508

File: src/robot_station_description/urdf/messzelle_new_macro.urdf.xacro (robot description, xacro)
@@ -150,5 +150,5 @@
             <parent link="${prefix}ct_load_block_link"/>
             <child link="${prefix}placement_link"/>
-            <origin xyz="0.0 0.16 0.15" rpy="0 -${pi/4} ${3*pi/2}" />
+            <origin xyz="0.0 0.16 0.17" rpy="0 -${2*pi/5} ${3*pi/2}" />
         </joint>
         <link name="${prefix}wall1_link">
