Commit message: Reques to merge dev branch to main (#5)
* Updated README to progress on 20260517

* Added AGV Table in description and moveit config

* Modified mqtt username and password to personal broker for test purpose

File: src/robot_station_description/urdf/orbbec_femto_mega_macro.urdf.xacro (robot description, xacro)
@@ -27,4 +27,11 @@
         </inertial>
     </link>
+    <link name="${prefix}camera_link" />
+    <joint name="${prefix}camera_joint" type="fixed">
+      <!-- The parent link must be read from the robot model it is attached to. -->
+      <parent link="${prefix}orbbec_femto_mega_link"/>
+      <child link="${prefix}camera_link"/>
+      <origin xyz="0 0 0" rpy="0 0 0"/>
+    </joint>
   </xacro:macro>
 </robot>

File: src/robot_station_description/urdf/station_800x440_bosch_macro.urdf.xacro (robot description, xacro)
@@ -6,5 +6,5 @@
           <origin xyz="0 0 0" rpy="0 0 0" />
           <geometry>
-            <box size="0.8 0.44 0.848"/>
+            <box size="0.8 0.44 0.859"/>
           </geometry>
           <material name="grey"/>
@@ -13,8 +13,8 @@
           <origin xyz="0 0 0" rpy="0 0 0"/>
           <geometry>
-            <box size="0.8 0.44 0.848"/>
+            <box size="0.8 0.44 0.859"/>
           </geometry>
         </collision>
-        <xacro:box_inertia m="150.0" x="0.8" y="0.44" z="0.848" o_xyz="0 0 0" o_rpy="0 0 0"/>
+        <xacro:box_inertia m="150.0" x="0.8" y="0.44" z="0.859" o_xyz="0 0 0" o_rpy="0 0 0"/>
     </link>
     <joint name="${prefix}station_800x440_base_joint" type="fixed">
@@ -22,5 +22,5 @@
       <parent link="${parent}"/>
       <child link="${prefix}robot_station_800x440_link"/>
-      <origin xyz="1.445 2.712 0.424" rpy="0 0 0"/>
+      <origin xyz="1.445 2.712 0.4295" rpy="0 0 0"/>
     </joint>
     <link name="${child}"/>
@@ -28,5 +28,5 @@
       <parent link="${prefix}robot_station_800x440_link"/>
       <child link="${child}"/>
-      <origin xyz="0 0 0.424" rpy="0 0 0"/>
+      <origin xyz="0 0 0.4295" rpy="0 0 0"/>
     </joint>
   </xacro:macro>

File: src/robot_station_description/urdf/station_ur_orbbec_robotiq2f140.urdf.xacro (robot description, xacro)
@@ -4,6 +4,8 @@
     <xacro:include filename="$(find robot_station_description)/urdf/common_properties.urdf"/>
     <xacro:include filename="$(find robot_station_description)/urdf/station_800x440_bosch_macro.urdf.xacro"/>
+    <xacro:include filename="$(find robot_station_description)/urdf/agv_station_550x400_macro.urdf.xacro"/>
     <xacro:include filename="$(find robot_station_description)/urdf/ur_orbbec_robotiq2f140_macro.urdf.xacro"/>
-    <xacro:include filename="$(find robot_station_description)/urdf/messzelle_macro.urdf.xacro"/>
+    <!-- <xacro:include filename="$(find robot_station_description)/urdf/messzelle_macro.urdf.xacro"/> -->
+    <xacro:include filename="$(find robot_station_description)/urdf/messzelle_new_macro.urdf.xacro"/>
     <!-- <xacro:include filename="$(find ifl_air_description)/urdf/robotertisch_1520x900_macro.urdf.xacro"/> -->
     <!-- <xacro:include filename="$(find ifl_air_description)/urdf/robotertisch_kameraaufsatz_macro.urdf.xacro"/> -->
@@ -15,7 +17,9 @@
     <!-- <xacro:arg name="joint_limit_params" default="$(find robot_station_cell_moveit_config)/config/joint_limits.yaml"/> -->
     <xacro:robot_station_800x440 prefix="" parent="world" child="table_mount_link"/>
+    <xacro:agv_station_550x400 prefix="" parent="world" />
     <xacro:ur_orbbec_robotiq prefix="" parent="table_mount_link" finger_type="default" mount_orbbec="true">
         <origin xyz="0 0 0" rpy="0 0 0"/>
     </xacro:ur_orbbec_robotiq>
-    <xacro:messzelle_env prefix="" parent="world"/>
+    <!-- <xacro:messzelle_env prefix="" parent="world"/> -->
+    <xacro:messzelle_env_new prefix="" parent="world"/>
 </robot>

File: src/robot_station_description/urdf/ur_orbbec_robotiq2f140_macro.urdf.xacro (robot description, xacro)
@@ -122,5 +122,5 @@
         <parent link="${prefix}tool0"/>
         <child link="tcp"/>
-        <origin xyz="0 0 0.18" rpy="0 0 0"/>
+        <origin xyz="0 0 0.24" rpy="0 0 0"/>
     </joint>
     <link name="tcp"/>
