Commit message: Connect camera links, Moved AGV table away for 25cm, New pose2 added in moveit config, Virtual joint for doors

File: src/robot_station_description/urdf/agv_station_550x400_macro.urdf.xacro (robot description, xacro)
@@ -22,5 +22,5 @@
       <parent link="${parent}"/>
       <child link="${prefix}station_agv_link"/>
-      <origin xyz="1.445 3.162 0.4725" rpy="0 0 0"/>
+      <origin xyz="1.445 3.412 0.4725" rpy="0 0 0"/>
     </joint>
     <link name="${prefix}agv_table_center_link"/>

Commit message: agv center link z+0.3, joint limit wrist3 -120~360

File: src/robot_station_description/urdf/agv_station_550x400_macro.urdf.xacro (robot description, xacro)
@@ -28,5 +28,5 @@
       <parent link="${prefix}station_agv_link"/>
       <child link="${prefix}agv_table_center_link"/>
-      <origin xyz="0 0 0.4875" rpy="0 0 0"/>
+      <origin xyz="0 0 0.5175" rpy="0 0 0"/>
     </joint>
   </xacro:macro>
