Commit message: tcp 0.24

File: src/robot_station_description/urdf/ur_orbbec_robotiq2f140_macro.urdf.xacro (robot description, xacro)
@@ -122,5 +122,5 @@
         <parent link="${prefix}tool0"/>
         <child link="tcp"/>
-        <origin xyz="0 0 0.23" rpy="0 0 0"/>
+        <origin xyz="0 0 0.24" rpy="0 0 0"/>
     </joint>
     <link name="tcp"/>

Commit message: New caliberation TCP

File: src/robot_station_description/urdf/ur_orbbec_robotiq2f140_macro.urdf.xacro (robot description, xacro)
@@ -122,5 +122,5 @@
         <parent link="${prefix}tool0"/>
         <child link="tcp"/>
-        <origin xyz="0 0 0.24" rpy="0 0 0"/>
+        <origin xyz="0 0.02 0.25" rpy="0 0 0"/>
     </joint>
     <link name="tcp"/>

Commit message: Updated README

File: src/robot_station_description/urdf/ur_orbbec_robotiq2f140_macro.urdf.xacro (robot description, xacro)
@@ -122,5 +122,5 @@
         <parent link="${prefix}tool0"/>
         <child link="tcp"/>
-        <origin xyz="0 0.02 0.25" rpy="0 0 0"/>
+        <origin xyz="0 -0.005 0.25" rpy="0 0 0"/>
     </joint>
     <link name="tcp"/>

Commit message: New caliberation TCP 20260605

File: src/robot_station_description/urdf/ur_orbbec_robotiq2f140_macro.urdf.xacro (robot description, xacro)
@@ -122,5 +122,5 @@
         <parent link="${prefix}tool0"/>
         <child link="tcp"/>
-        <origin xyz="0 -0.005 0.25" rpy="0 0 0"/>
+        <origin xyz="0 0 0.25" rpy="0 0 0"/>
     </joint>
     <link name="tcp"/>
